File: boards/loggerboard.kicad_sch (KiCad schematic)
At the start: 23 parts, among them J2 Micro_SD_Card, J7 RS485_logger_2, J8 RS485_logger, J9 BNO085, U2 MAX3485, U5 MOUDLE-SEEEDUINO-XIAO-ESP32C3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, U6 DS3231MZ

Commit message: 増幅回路追加
Parts:
- C2: footprint Capacitor_SMD:C_0603_1608Metric_Pad1.08x0.95mm_HandSolder -> Capacitor_SMD:C_1210_3225Metric_Pad1.33x2.70mm_HandSolder
Changed lines of the file:
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@@
 			)
 		)
-		(property "Footprint" "Capacitor_SMD:C_0603_1608Metric_Pad1.08x0.95mm_HandSolder"
+		(property "Footprint" "Capacitor_SMD:C_1210_3225Metric_Pad1.33x2.70mm_HandSolder"
 			(at 162.56 152.4 0)
 			(effects
