File: boards/TFTboard.kicad_sch (KiCad schematic)
At the start: 27 parts, among them J1 5051104096, J10 Conn_01x04, J13 Conn_01x03 speaker, J3 URM37, J4 Conn_01x03 servo, J5 RS485_TFT, J6 Conn_01x03 encoder_direct, SW1 SW_DIP_x01, U1 MOUDLE-SEEEDUINO-XIAO-ESP32C3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, U11 MOUDLE-SEEEDUINO-XIAO-ESP32C3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

Commit message: DRCエラー解消
Parts:
- J4: value Conn_01x03 servo -> servo
- J6: value Conn_01x03 encoder_direct -> encoder_direct
Changed lines of the file:
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@@
 			)
 		)
-		(property "Value" "Conn_01x03 servo"
+		(property "Value" "servo"
 			(at 148.59 95.2499 0)
 			(effects
@@
 			)
 		)
-		(property "Value" "Conn_01x03 encoder_direct"
+		(property "Value" "encoder_direct"
 			(at 148.59 105.4099 0)
 			(effects
